File: PCB/PCB.sch (KiCad schematic (older format))
At the start: 18 parts, among them J1 Conn_01x04_Female, J2 Conn_01x04_Female, J3 Conn_01x04_Female, J4 Conn_01x04_Female, J5 MiniMicroJst2.0Ph3Pin, J6 Conn_01x02_Female, J7 Conn_01x02_Female, U1 ESP01, U2 MicroSDCardModule

Commit message: bugfixing
Parts:
- added R7: R, Resistor_THT:R_Axial_DIN0411_L9.9mm_D3.6mm_P12.70mm_Horizontal, symbol Device:R
- added SW1: SW_Push, Button_Switch_THT:SW_PUSH_6mm, symbol Switch:SW_Push
Connections:
- net +3V3: now also A3.4 (3V3), SW1.1
- net GND: now also A3.29 (GND), A3.7 (GND), R7.1
- net at U1.4 (GPIO2): now also R7.2, SW1.2
- no-connect marks 25 -> 21
Changed lines of the file:
@@
 L power:GND #PWR0113
 U 1 1 5E32B94F
-P 1400 2450
-F 0 "#PWR0113" H 1400 2200 50  0001 C CNN
-F 1 "GND" H 1405 2277 50  0000 C CNN
-F 2 "" H 1400 2450 50  0001 C CNN
-F 3 "" H 1400 2450 50  0001 C CNN
-	1    1400 2450
+P 1400 2550
+F 0 "#PWR0113" H 1400 2300 50  0001 C CNN
+F 1 "GND" H 1405 2377 50  0000 C CNN
+F 2 "" H 1400 2550 50  0001 C CNN
+F 3 "" H 1400 2550 50  0001 C CNN
+	1    1400 2550
 	1    0    0    -1
 $EndComp
@@
 Wire Wire Line
 	2350 1550 2400 1550
-$Comp
-L My_Library:ESP01 U1
-U 1 1 5E315A39
-P 1850 850
-F 0 "U1" H 1825 915 50  0000 C CNN
-F 1 "ESP01" H 1825 824 50  0000 C CNN
-F 2 "ESP8266:ESP-01" H 2000 800 50  0001 C CNN
-F 3 "" H 2000 800 50  0001 C CNN
-	1    1850 850
-	1    0    0    -1
-$EndComp
 NoConn ~ 2250 1400
 NoConn ~ 1400 1400
-NoConn ~ 1400 1250
 $Comp
 L power:GND #PWR0115
@@
 L power:GND #PWR0120
 U 1 1 5E338518
-P 5350 3250
-F 0 "#PWR0120" H 5350 3000 50  0001 C CNN
-F 1 "GND" H 5355 3077 50  0000 C CNN
-F 2 "" H 5350 3250 50  0001 C CNN
-F 3 "" H 5350 3250 50  0001 C CNN
-	1    5350 3250
+P 5350 3350
+F 0 "#PWR0120" H 5350 3100 50  0001 C CNN
+F 1 "GND" H 5355 3177 50  0000 C CNN
+F 2 "" H 5350 3350 50  0001 C CNN
+F 3 "" H 5350 3350 50  0001 C CNN
+	1    5350 3350
 	1    0    0    -1
 $EndComp
@@
 L power:VCC #PWR0123
 U 1 1 5E368F72
-P 5550 1150
-F 0 "#PWR0123" H 5550 1000 50  0001 C CNN
-F 1 "VCC" H 5568 1323 50  0000 C CNN
-F 2 "" H 5550 1150 50  0001 C CNN
-F 3 "" H 5550 1150 50  0001 C CNN
-	1    5550 1150
+P 5550 900
+F 0 "#PWR0123" H 5550 750 50  0001 C CNN
+F 1 "VCC" H 5568 1073 50  0000 C CNN
+F 2 "" H 5550 900 50  0001 C CNN
+F 3 "" H 5550 900 50  0001 C CNN
+	1    5550 900
 	1    0    0    -1
 $EndComp
@@
 Wire Wire Line
 	4550 2450 4850 2450
-NoConn ~ 5250 3250
-NoConn ~ 5450 3250
 Connection ~ 7150 1850
 $Comp
@@
 $EndComp
 NoConn ~ 5250 1150
-NoConn ~ 5450 1150
 $Comp
 L Device:R R5
@@
 	-1   0    0    1
 $EndComp
+Wire Wire Line
+	1400 2550 1400 2500
+$Comp
+L Switch:SW_Push SW1
+U 1 1 5E5EB1BE
+P 1000 1750
+F 0 "SW1" H 1000 2035 50  0000 C CNN
+F 1 "SW_Push" H 1000 1944 50  0000 C CNN
+F 2 "Button_Switch_THT:SW_PUSH_6mm" H 1000 1950 50  0001 C CNN
+F 3 "~" H 1000 1950 50  0001 C CNN
+	1    1000 1750
+	1    0    0    -1
+$EndComp
+Wire Wire Line
+	1250 1750 1200 1750
+Connection ~ 1400 2500
+Wire Wire Line
+	1400 2500 1400 2450
+Wire Wire Line
+	1250 1750 1250 1250
+Wire Wire Line
+	1250 1250 1400 1250
+$Comp
+L My_Library:ESP01 U1
+U 1 1 5E315A39
+P 1850 850
+F 0 "U1" H 1825 915 50  0000 C CNN
+F 1 "ESP01" H 1825 824 50  0000 C CNN
+F 2 "ESP8266:ESP-01" H 2000 800 50  0001 C CNN
+F 3 "" H 2000 800 50  0001 C CNN
+	1    1850 850
+	1    0    0    -1
+$EndComp
+$Comp
+L power:+3.3V #PWR0126
+U 1 1 5E5F3476
+P 750 1050
+F 0 "#PWR0126" H 750 900 50  0001 C CNN
+F 1 "+3.3V" V 765 1178 50  0000 L CNN
+F 2 "" H 750 1050 50  0001 C CNN
+F 3 "" H 750 1050 50  0001 C CNN
+	1    750  1050
+	1    0    0    -1
+$EndComp
+Wire Wire Line
+	800  1750 750  1750
+Wire Wire Line
+	750  1750 750  1050
+Wire Wire Line
+	5350 3250 5350 3300
+Wire Wire Line
+	5350 3300 5250 3300
+Wire Wire Line
+	5250 3300 5250 3250
+Connection ~ 5350 3300
+Wire Wire Line
+	5350 3300 5350 3350
+Wire Wire Line
+	5350 3300 5450 3300
+Wire Wire Line
+	5450 3300 5450 3250
+Wire Wire Line
+	5550 900  5550 1150
+$Comp
+L power:+3.3V #PWR0127
+U 1 1 5E6068AC
+P 5450 850
+F 0 "#PWR0127" H 5450 700 50  0001 C CNN
+F 1 "+3.3V" V 5465 978 50  0000 L CNN
+F 2 "" H 5450 850 50  0001 C CNN
+F 3 "" H 5450 850 50  0001 C CNN
+	1    5450 850
+	1    0    0    -1
+$EndComp
+Wire Wire Line
+	5450 850  5450 1150
+$Comp
+L Device:R R7
+U 1 1 5E6112B8
+P 1250 2300
+F 0 "R7" H 1300 2250 50  0000 L CNN
+F 1 "R" H 1350 2250 50  0000 L CNN
+F 2 "Resistor_THT:R_Axial_DIN0411_L9.9mm_D3.6mm_P12.70mm_Horizontal" V 1180 2300 50  0001 C CNN
+F 3 "~" H 1250 2300 50  0001 C CNN
+	1    1250 2300
+	-1   0    0    1
+$EndComp
+Wire Wire Line
+	1250 2500 1250 2450
+Wire Wire Line
+	1250 2500 1400 2500
+Wire Wire Line
+	1250 2150 1250 1750
+Connection ~ 1250 1750
 $EndSCHEMATC
